File: Plant-guardian.kicad_pcb (KiCad board)
At the start: 2 copper layers, 74.5 x 91 mm, 80 parts, among them J1 USB_C_Receptacle_USB2.0_16P, J2 Conn_01x02_Pin, J3 Conn_01x02_Pin, J4 Conn_01x03_Pin, Q1 SS8050, Q2 SS8050, Q3 HKTD90N03, Q4 HKTD90N03, SW1 KMR221GLFS, SW2 KMR221GLFS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

Commit message: rev0 ready
Parts:
- added G***: LOGO, LOGO, F.Cu at (112.6, 131.3)
- added G***: LOGO, LOGO, B.Cu at (76.9, 129.8)
- added G***: LOGO, LOGO, B.Cu at (114.7, 87.5)
- added G***: LOGO, LOGO, B.Cu at (106.8, 109.1)
- added G***: LOGO, LOGO, B.Cu at (107.3, 131.7)
- added J5: Conn_01x03_Pin, Connector_PinHeader_2.54mm:PinHeader_1x03_P2.54mm_Vertical, F.Cu at (115.8, 115.6)
- added kibuzzard-691EE203: G***, kibuzzard-691EE203, F.Cu at (105.8, 131.0)
- moved R16 10.7 mm to (110.2, 63.8)
- moved D4 5.67 mm to (108.9, 59.3), turned to 0 degrees
- moved D3 5.41 mm to (103.3, 59.3), turned to 0 degrees
- moved C18 5.09 mm to (103.6, 62.8), turned to 180 degrees
- moved C24 3.68 mm to (103.5, 72.5), turned to 180 degrees
- moved C25 3.68 mm to (103.5, 65.3), turned to 180 degrees
- moved J2 3.68 mm to (103.7, 74.8)
- moved J3 3.68 mm to (103.7, 67.6)
- moved Q3 3.68 mm to (97.0, 75.8)
- moved Q4 3.68 mm to (97.0, 68.5)
- moved R19 3.68 mm to (90.0, 75.5)
- moved R20 3.68 mm to (90.0, 73.5)
- moved R25 3.68 mm to (90.0, 68.1)
- moved R27 3.68 mm to (90.0, 66.1)
- moved C13 0.22 mm to (125.0, 104.5)
Connections:
- DD1 pad 10: unconnected-(DD1-IO25-Pad10) -> PUMP
- DD1 pad 11: unconnected-(DD1-IO26-Pad11) -> FAN
- DD1 pad 24: RS -> unconnected-(DD1-IO2-Pad24)
- DD1 pad 26: RES -> unconnected-(DD1-IO4-Pad26)
- DD1 pad 27: unconnected-(DD1-IO16-Pad27) -> !SS
- DD1 pad 28: unconnected-(DD1-IO17-Pad28) -> RES
- DD1 pad 29: !SS -> unconnected-(DD1-IO5-Pad29)
- DD1 pad 31: unconnected-(DD1-IO19-Pad31) -> RS
Routing:
- net 3.3V: track 0.00 -> 120.3 mm, vias 0 -> 18
- net LED_CNTRL: track 0.00 -> 91.7 mm, vias 0 -> 2
- net SDA: track 0.00 -> 60.1 mm, vias 0 -> 2
- net PUMP: track 0.00 -> 57.0 mm
- net SCL: track 0.00 -> 51.3 mm, vias 0 -> 2
- net FAN: track 0.00 -> 49.7 mm
- net TX: track 0.31 -> 32.0 mm, vias 1 -> 2
- net !RST: track 6.87 -> 37.5 mm, vias 0 -> 2
- net RX: track 0.31 -> 29.6 mm, vias 1 -> 2
- net !SS: track 0.00 -> 27.6 mm, vias 0 -> 1
- net SENSOR_OUT: track 1.72 -> 29.2 mm
- net SCLK: track 0.00 -> 22.4 mm, vias 0 -> 1
- net RS: track 0.00 -> 21.7 mm, vias 0 -> 1
- net RES: track 0.00 -> 20.0 mm, vias 0 -> 1
- net GPIO 0: track 3.74 -> 20.0 mm, vias 0 -> 2
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- added copper zone on F.Cu, net 12V
- added copper zone on B.Cu, net 3.3V
- added copper zone on F.Cu, net 3.3V
- added copper zone on B.Cu, net 5V
- added copper zone on F.Cu, net 5V
- added copper zone on B.Cu, net Earth
- added copper zone on F.Cu, net Earth
- added copper zone on F.Cu, net Net-(D1-A)
- added copper zone on F.Cu, net Net-(J2-Pin_2)
- added copper zone on F.Cu, net Net-(J3-Pin_2)
Other:
- board text added: "12V"
- board text added: "Fans"
- board text added: "GND"
- board text added: "Pump"
- board text added: "by @madjogger"
